Commit message: changed the xacro and fleet_brain, added single_brain

File: src/vector_agv_v2/urdf/vector_v2.urdf.xacro (robot description, xacro)
@@ -76,13 +76,17 @@
       <axis xyz="0 1 0"/>
     </joint>
+    <gazebo reference="${prefix}_wheel">
+      <mu1>1.0</mu1>
+      <mu2>1.0</mu2>
+    </gazebo>
   </xacro:macro>
   <xacro:macro name="caster_wheel" params="prefix x_offset y_offset">
     <link name="${prefix}_wheel">
       <visual>
-        <geometry><sphere radius="0.2"/></geometry>
+        <geometry><sphere radius="0.19"/></geometry>
         <material name="pu_orange"><color rgba="1.0 0.4 0.0 1.0"/></material>
       </visual>
       <collision>
-        <geometry><sphere radius="0.2"/></geometry>
+        <geometry><sphere radius="0.19"/></geometry>
       </collision>
       <inertial>
@@ -96,4 +100,8 @@
       <origin xyz="${x_offset} ${y_offset} -0.2" rpy="0 0 0"/>
     </joint>
+    <gazebo reference="${prefix}_wheel">
+      <mu1>0.0</mu1>
+      <mu2>0.0</mu2>
+    </gazebo>
   </xacro:macro>
   <xacro:drive_wheel prefix="drive_left" y_offset="0.45"/>
@@ -118,5 +126,6 @@
       <update_rate>10.0</update_rate>
       <camera>
-        <horizontal_fov>2.0</horizontal_fov> <image>
+        <horizontal_fov>2.0</horizontal_fov>
+        <image>
           <width>160</width>
           <height>120</height>
@@ -138,7 +147,3 @@
     </plugin>
   </gazebo>
-  <gazebo reference="front_left_wheel"><mu1>0.0</mu1><mu2>0.0</mu2></gazebo>
-  <gazebo reference="front_right_wheel"><mu1>0.0</mu1><mu2>0.0</mu2></gazebo>
-  <gazebo reference="rear_left_wheel"><mu1>0.0</mu1><mu2>0.0</mu2></gazebo>
-  <gazebo reference="rear_right_wheel"><mu1>0.0</mu1><mu2>0.0</mu2></gazebo>
 </robot>

Commit message: single_brain works perfectly

File: src/vector_agv_v2/urdf/vector_v2.urdf.xacro (robot description, xacro)
@@ -120,5 +120,5 @@
     <parent link="base_link"/>
     <child link="camera_link"/>
-    <origin xyz="1.5 0 0.8" rpy="0 1.5708 0"/>
+    <origin xyz="4.3 0 0.8" rpy="0 1.5708 0"/>
   </joint>
   <gazebo reference="camera_link">

Commit message: fleet_logic restored - no fishtailing just understeer

File: src/vector_agv_v2/urdf/vector_v2.urdf.xacro (robot description, xacro)
@@ -25,4 +25,5 @@
     </collision>
     <inertial>
+      <origin xyz="0 0 -0.5" rpy="0 0 0"/>
       <mass value="500.0"/>
       <inertia ixx="71.0" ixy="0.0" ixz="0.0" iyy="2344.0" iyz="0.0" izz="2414.0"/>
@@ -40,4 +41,5 @@
     </collision>
     <inertial>
+      <origin xyz="0 0 -1.5" rpy="0 0 0"/>
       <mass value="${payload_mass}"/>
       <inertia
@@ -126,5 +128,5 @@
       <update_rate>10.0</update_rate>
       <camera>
-        <horizontal_fov>2.0</horizontal_fov>
+        <horizontal_fov>2.5</horizontal_fov>
         <image>
           <width>160</width>
@@ -142,4 +144,6 @@
       <wheel_radius>0.2</wheel_radius>
       <topic>/${ns}/cmd_vel</topic>
+      <max_linear_acceleration>10.0</max_linear_acceleration>
+      <max_angular_acceleration>20.0</max_angular_acceleration>
     </plugin>
     <plugin filename="gz-sim-joint-state-publisher-system" name="gz::sim::systems::JointStatePublisher">

Commit message: changed agv to match requirements

File: src/vector_agv_v2/urdf/vector_v2.urdf.xacro (robot description, xacro)
@@ -4,19 +4,15 @@
   <xacro:property name="ns" value="$(arg namespace)"/>
   <xacro:property name="payload_mass" value="2000.0"/>
+  <material name="heavy_orange">
+    <color rgba="1.0 0.45 0.0 1.0"/>
+  </material>
+  <material name="steel">
+    <color rgba="0.6 0.6 0.65 1.0"/>
+  </material>
   <link name="base_link">
     <visual>
       <origin xyz="0 0 0" rpy="0 0 0"/>
-      <geometry><box size="7.0 1.3 0.15"/></geometry>
-      <material name="off_white"><color rgba="0.9 0.9 0.9 1.0"/></material>
-    </visual>
-    <visual>
-      <origin xyz="3.5 0 0" rpy="0 0 0"/>
-      <geometry><cylinder radius="0.65" length="0.15"/></geometry>
-      <material name="off_white"><color rgba="0.9 0.9 0.9 1.0"/></material>
-    </visual>
-    <visual>
-      <origin xyz="-3.5 0 0" rpy="0 0 0"/>
-      <geometry><cylinder radius="0.65" length="0.15"/></geometry>
-      <material name="off_white"><color rgba="0.9 0.9 0.9 1.0"/></material>
+      <geometry><box size="7.5 1.3 0.25"/></geometry>
+      <material name="heavy_orange"/>
     </visual>
     <collision>
@@ -30,10 +26,54 @@
     </inertial>
   </link>
+  <xacro:macro name="rod_column" params="x_val">
+    <visual><origin xyz="${x_val} 0 0.5" rpy="1.5708 0 0"/><geometry><cylinder radius="0.03" length="1.2"/></geometry><material name="steel"/></visual>
+    <visual><origin xyz="${x_val} 0 0.8" rpy="1.5708 0 0"/><geometry><cylinder radius="0.03" length="1.2"/></geometry><material name="steel"/></visual>
+    <visual><origin xyz="${x_val} 0 1.1" rpy="1.5708 0 0"/><geometry><cylinder radius="0.03" length="1.2"/></geometry><material name="steel"/></visual>
+    <visual><origin xyz="${x_val} 0 1.4" rpy="1.5708 0 0"/><geometry><cylinder radius="0.03" length="1.2"/></geometry><material name="steel"/></visual>
+    <visual><origin xyz="${x_val} 0 1.7" rpy="1.5708 0 0"/><geometry><cylinder radius="0.03" length="1.2"/></geometry><material name="steel"/></visual>
+    <visual><origin xyz="${x_val} 0 2.0" rpy="1.5708 0 0"/><geometry><cylinder radius="0.03" length="1.2"/></geometry><material name="steel"/></visual>
+  </xacro:macro>
   <link name="payload_link">
     <visual>
-      <origin xyz="0 0 1.25" rpy="0 0 0"/>
-      <geometry><box size="7.0 1.5 2.5"/></geometry>
-      <material name="dark_grey"><color rgba="0.3 0.3 0.3 1.0"/></material>
+      <origin xyz="3.0 0.5 0.15" rpy="0 0 0"/>
+      <geometry><box size="0.15 0.15 0.3"/></geometry>
+      <material name="steel"/>
     </visual>
+    <visual>
+      <origin xyz="3.0 -0.5 0.15" rpy="0 0 0"/>
+      <geometry><box size="0.15 0.15 0.3"/></geometry>
+      <material name="steel"/>
+    </visual>
+    <visual>
+      <origin xyz="-3.0 0.5 0.15" rpy="0 0 0"/>
+      <geometry><box size="0.15 0.15 0.3"/></geometry>
+      <material name="steel"/>
+    </visual>
+    <visual>
+      <origin xyz="-3.0 -0.5 0.15" rpy="0 0 0"/>
+      <geometry><box size="0.15 0.15 0.3"/></geometry>
+      <material name="steel"/>
+    </visual>
+    <visual>
+      <origin xyz="0 0 0.325" rpy="0 0 0"/>
+      <geometry><box size="7.0 1.3 0.05"/></geometry>
+      <material name="steel"/>
+    </visual>
+    <visual>
+      <origin xyz="0 0.6 1.25" rpy="0 0 0"/>
+      <geometry><box size="7.0 0.1 1.8"/></geometry>
+      <material name="steel"/>
+    </visual>
+    <xacro:rod_column x_val="-3.0"/>
+    <xacro:rod_column x_val="-2.4"/>
+    <xacro:rod_column x_val="-1.8"/>
+    <xacro:rod_column x_val="-1.2"/>
+    <xacro:rod_column x_val="-0.6"/>
+    <xacro:rod_column x_val="0.0"/>
+    <xacro:rod_column x_val="0.6"/>
+    <xacro:rod_column x_val="1.2"/>
+    <xacro:rod_column x_val="1.8"/>
+    <xacro:rod_column x_val="2.4"/>
+    <xacro:rod_column x_val="3.0"/>
     <collision>
       <origin xyz="0 0 1.25" rpy="0 0 0"/>

Commit message: added lights

File: src/vector_agv_v2/urdf/vector_v2.urdf.xacro (robot description, xacro)
@@ -4,10 +4,9 @@
   <xacro:property name="ns" value="$(arg namespace)"/>
   <xacro:property name="payload_mass" value="2000.0"/>
-  <material name="heavy_orange">
-    <color rgba="1.0 0.45 0.0 1.0"/>
-  </material>
-  <material name="steel">
-    <color rgba="0.6 0.6 0.65 1.0"/>
-  </material>
+  <material name="heavy_orange"><color rgba="1.0 0.45 0.0 1.0"/></material>
+  <material name="steel"><color rgba="0.6 0.6 0.65 1.0"/></material>
+  <material name="industrial_black"><color rgba="0.1 0.1 0.1 1.0"/></material>
+  <material name="headlight_white"><color rgba="1.0 1.0 1.0 1.0"/></material>
+  <material name="taillight_red"><color rgba="1.0 0.0 0.0 1.0"/></material>
   <link name="base_link">
     <visual>
@@ -15,4 +14,24 @@
       <geometry><box size="7.5 1.3 0.25"/></geometry>
       <material name="heavy_orange"/>
+    </visual>
+    <visual>
+      <origin xyz="3.76 0.45 0.05" rpy="0 0 0"/>
+      <geometry><box size="0.02 0.25 0.08"/></geometry>
+      <material name="headlight_white"/>
+    </visual>
+    <visual>
+      <origin xyz="3.76 -0.45 0.05" rpy="0 0 0"/>
+      <geometry><box size="0.02 0.25 0.08"/></geometry>
+      <material name="headlight_white"/>
+    </visual>
+    <visual>
+      <origin xyz="-3.76 0.45 0.05" rpy="0 0 0"/>
+      <geometry><box size="0.02 0.25 0.08"/></geometry>
+      <material name="taillight_red"/>
+    </visual>
+    <visual>
+      <origin xyz="-3.76 -0.45 0.05" rpy="0 0 0"/>
+      <geometry><box size="0.02 0.25 0.08"/></geometry>
+      <material name="taillight_red"/>
     </visual>
     <collision>
@@ -101,5 +120,5 @@
         <origin xyz="0 0 0" rpy="1.5708 0 0"/>
         <geometry><cylinder radius="0.2" length="0.1"/></geometry>
-        <material name="pu_orange"><color rgba="1.0 0.4 0.0 1.0"/></material>
+        <material name="industrial_black"/>
       </visual>
       <collision>
@@ -121,4 +140,5 @@
       <mu1>1.0</mu1>
       <mu2>1.0</mu2>
+      <material>Gazebo/DarkGrey</material>
     </gazebo>
   </xacro:macro>
@@ -127,5 +147,5 @@
       <visual>
         <geometry><sphere radius="0.19"/></geometry>
-        <material name="pu_orange"><color rgba="1.0 0.4 0.0 1.0"/></material>
+        <material name="industrial_black"/>
       </visual>
       <collision>
@@ -145,4 +165,5 @@
       <mu1>0.0</mu1>
       <mu2>0.0</mu2>
+      <material>Gazebo/DarkGrey</material>
     </gazebo>
   </xacro:macro>

Commit message: added siren

File: src/vector_agv_v2/urdf/vector_v2.urdf.xacro (robot description, xacro)
@@ -9,4 +9,7 @@
   <material name="headlight_white"><color rgba="1.0 1.0 1.0 1.0"/></material>
   <material name="taillight_red"><color rgba="1.0 0.0 0.0 1.0"/></material>
+  <material name="beacon_yellow"><color rgba="1.0 0.8 0.0 1.0"/></material>
+  <material name="button_red"><color rgba="0.8 0.1 0.1 1.0"/></material>
+  <material name="button_green"><color rgba="0.1 0.8 0.1 1.0"/></material>
   <link name="base_link">
     <visual>
@@ -83,4 +86,29 @@
       <geometry><box size="7.0 0.1 1.8"/></geometry>
       <material name="steel"/>
+    </visual>
+    <visual>
+      <origin xyz="-3.55 0.66 1.4" rpy="0 0 0"/>
+      <geometry><box size="0.1 0.25 0.4"/></geometry>
+      <material name="industrial_black"/>
+    </visual>
+    <visual>
+      <origin xyz="-3.61 0.66 1.48" rpy="0 1.5708 0"/>
+      <geometry><cylinder radius="0.05" length="0.04"/></geometry>
+      <material name="button_red"/>
+    </visual>
+    <visual>
+      <origin xyz="-3.61 0.66 1.32" rpy="0 1.5708 0"/>
+      <geometry><cylinder radius="0.03" length="0.03"/></geometry>
+      <material name="button_green"/>
+    </visual>
+    <visual>
+      <origin xyz="-3.4 0.6 2.3" rpy="0 0 0"/>
+      <geometry><cylinder radius="0.025" length="0.4"/></geometry>
+      <material name="industrial_black"/>
+    </visual>
+    <visual>
+      <origin xyz="-3.4 0.6 2.55" rpy="0 0 0"/>
+      <geometry><cylinder radius="0.07" length="0.12"/></geometry>
+      <material name="beacon_yellow"/>
     </visual>
     <xacro:rod_column x_val="-3.0"/>

Commit message: added siren better version

File: src/vector_agv_v2/urdf/vector_v2.urdf.xacro (robot description, xacro)
@@ -57,58 +57,17 @@
   </xacro:macro>
   <link name="payload_link">
-    <visual>
-      <origin xyz="3.0 0.5 0.15" rpy="0 0 0"/>
-      <geometry><box size="0.15 0.15 0.3"/></geometry>
-      <material name="steel"/>
-    </visual>
-    <visual>
-      <origin xyz="3.0 -0.5 0.15" rpy="0 0 0"/>
-      <geometry><box size="0.15 0.15 0.3"/></geometry>
-      <material name="steel"/>
-    </visual>
-    <visual>
-      <origin xyz="-3.0 0.5 0.15" rpy="0 0 0"/>
-      <geometry><box size="0.15 0.15 0.3"/></geometry>
-      <material name="steel"/>
-    </visual>
-    <visual>
-      <origin xyz="-3.0 -0.5 0.15" rpy="0 0 0"/>
-      <geometry><box size="0.15 0.15 0.3"/></geometry>
-      <material name="steel"/>
-    </visual>
-    <visual>
-      <origin xyz="0 0 0.325" rpy="0 0 0"/>
-      <geometry><box size="7.0 1.3 0.05"/></geometry>
-      <material name="steel"/>
-    </visual>
-    <visual>
-      <origin xyz="0 0.6 1.25" rpy="0 0 0"/>
-      <geometry><box size="7.0 0.1 1.8"/></geometry>
-      <material name="steel"/>
-    </visual>
-    <visual>
-      <origin xyz="-3.55 0.66 1.4" rpy="0 0 0"/>
-      <geometry><box size="0.1 0.25 0.4"/></geometry>
-      <material name="industrial_black"/>
-    </visual>
-    <visual>
-      <origin xyz="-3.61 0.66 1.48" rpy="0 1.5708 0"/>
-      <geometry><cylinder radius="0.05" length="0.04"/></geometry>
-      <material name="button_red"/>
-    </visual>
-    <visual>
-      <origin xyz="-3.61 0.66 1.32" rpy="0 1.5708 0"/>
-      <geometry><cylinder radius="0.03" length="0.03"/></geometry>
-      <material name="button_green"/>
-    </visual>
+    <visual><origin xyz="3.0 0.5 0.15" rpy="0 0 0"/><geometry><box size="0.15 0.15 0.3"/></geometry><material name="steel"/></visual>
+    <visual><origin xyz="3.0 -0.5 0.15" rpy="0 0 0"/><geometry><box size="0.15 0.15 0.3"/></geometry><material name="steel"/></visual>
+    <visual><origin xyz="-3.0 0.5 0.15" rpy="0 0 0"/><geometry><box size="0.15 0.15 0.3"/></geometry><material name="steel"/></visual>
+    <visual><origin xyz="-3.0 -0.5 0.15" rpy="0 0 0"/><geometry><box size="0.15 0.15 0.3"/></geometry><material name="steel"/></visual>
+    <visual><origin xyz="0 0 0.325" rpy="0 0 0"/><geometry><box size="7.0 1.3 0.05"/></geometry><material name="steel"/></visual>
+    <visual><origin xyz="0 0.6 1.25" rpy="0 0 0"/><geometry><box size="7.0 0.1 1.8"/></geometry><material name="steel"/></visual>
+    <visual><origin xyz="-3.55 0.66 1.4" rpy="0 0 0"/><geometry><box size="0.1 0.25 0.4"/></geometry><material name="industrial_black"/></visual>
+    <visual><origin xyz="-3.61 0.66 1.48" rpy="0 1.5708 0"/><geometry><cylinder radius="0.05" length="0.04"/></geometry><material name="button_red"/></visual>
+    <visual><origin xyz="-3.61 0.66 1.32" rpy="0 1.5708 0"/><geometry><cylinder radius="0.03" length="0.03"/></geometry><material name="button_green"/></visual>
     <visual>
       <origin xyz="-3.4 0.6 2.3" rpy="0 0 0"/>
       <geometry><cylinder radius="0.025" length="0.4"/></geometry>
       <material name="industrial_black"/>
-    </visual>
-    <visual>
-      <origin xyz="-3.4 0.6 2.55" rpy="0 0 0"/>
-      <geometry><cylinder radius="0.07" length="0.12"/></geometry>
-      <material name="beacon_yellow"/>
     </visual>
     <xacro:rod_column x_val="-3.0"/>
@@ -131,8 +90,6 @@
       <mass value="${payload_mass}"/>
       <inertia
-        ixx="${(payload_mass/12.0) * (1.5*1.5 + 2.5*2.5)}"
-        ixy="0.0" ixz="0.0"
-        iyy="${(payload_mass/12.0) * (7.0*7.0 + 2.5*2.5)}"
-        iyz="0.0"
+        ixx="${(payload_mass/12.0) * (1.5*1.5 + 2.5*2.5)}" ixy="0.0" ixz="0.0"
+        iyy="${(payload_mass/12.0) * (7.0*7.0 + 2.5*2.5)}" iyz="0.0"
         izz="${(payload_mass/12.0) * (7.0*7.0 + 1.5*1.5)}"/>
     </inertial>
@@ -143,4 +100,58 @@
     <origin xyz="0 0 0.075" rpy="0 0 0"/>
   </joint>
+  <link name="beacon_link">
+    <visual>
+      <origin xyz="0 0 0.06" rpy="0 0 0"/>
+      <geometry><cylinder radius="0.07" length="0.12"/></geometry>
+      <material name="beacon_yellow"/>
+    </visual>
+    <inertial>
+      <mass value="0.05"/>
+      <inertia ixx="0.0001" ixy="0" ixz="0" iyy="0.0001" iyz="0" izz="0.0001"/>
+    </inertial>
+  </link>
+  <joint name="beacon_joint" type="continuous">
+    <parent link="payload_link"/>
+    <child link="beacon_link"/>
+    <origin xyz="-3.4 0.6 2.5" rpy="0 0 0"/>
+    <axis xyz="0 0 1"/>
+  </joint>
+  <gazebo reference="beacon_link">
+    <material>Gazebo/Yellow</material>
+    <light name="siren_beam_1" type="spot">
+      <pose>0 0 0.06 0 1.5708 0</pose>
+      <diffuse>1.0 0.8 0.0 1.0</diffuse>
+      <specular>1.0 0.8 0.0 1.0</specular>
+      <attenuation>
+        <range>10.0</range>
+        <linear>0.1</linear>
+        <constant>0.1</constant>
+        <quadratic>0.01</quadratic>
+      </attenuation>
+      <spot>
+        <inner_angle>0.2</inner_angle>
+        <outer_angle>1.0</outer_angle>
+        <falloff>1.0</falloff>
+      </spot>
+      <cast_shadows>false</cast_shadows>
+    </light>
+    <light name="siren_beam_2" type="spot">
+      <pose>0 0 0.06 0 -1.5708 0</pose>
+      <diffuse>1.0 0.8 0.0 1.0</diffuse>
+      <specular>1.0 0.8 0.0 1.0</specular>
+      <attenuation>
+        <range>10.0</range>
+        <linear>0.1</linear>
+        <constant>0.1</constant>
+        <quadratic>0.01</quadratic>
+      </attenuation>
+      <spot>
+        <inner_angle>0.2</inner_angle>
+        <outer_angle>1.0</outer_angle>
+        <falloff>1.0</falloff>
+      </spot>
+      <cast_shadows>false</cast_shadows>
+    </light>
+  </gazebo>
   <xacro:macro name="drive_wheel" params="prefix y_offset">
     <link name="${prefix}_wheel">
@@ -218,8 +229,5 @@
       <camera>
         <horizontal_fov>2.5</horizontal_fov>
-        <image>
-          <width>160</width>
-          <height>120</height>
-        </image>
+        <image><width>160</width><height>120</height></image>
       </camera>
       <topic>/${ns}/camera/image_raw</topic>
@@ -236,7 +244,13 @@
       <max_angular_acceleration>20.0</max_angular_acceleration>
     </plugin>
-    <plugin filename="gz-sim-joint-state-publisher-system" name="gz::sim::systems::JointStatePublisher">
-      <topic>/${ns}/joint_states</topic>
+    <plugin filename="libgz-sim-joint-velocity-controller-system.so" name="gz::sim::systems::JointVelocityController">
+      <joint_name>beacon_joint</joint_name>
+      <topic>/${ns}/beacon_spin</topic>
+      <initial_velocity>15.0</initial_velocity>
     </plugin>
+    <plugin filename="gz-sim-joint-velocity-controller-system" name="gz::sim::systems::JointVelocityController">
+      <joint_name>beacon_joint</joint_name>
+      <topic>/${ns}/beacon_spin</topic>
+      <initial_velocity>15.0</initial_velocity> </plugin>
   </gazebo>
 </robot>
